File: MPSIBOARD/MPSIBOARD.sch (KiCad schematic (older format))
At the start: 60 parts, among them J1 9830 IO CONN, J2 USB_B_Mini, J3 Micro_SD_Card_Det_Hirose_DM3AT, J4 Xilinx-JTAG, J5 STM32-JTAG, U1 XC2C32A, U10 74LS38, U11 AMS1117-3.3, U2 STM32F407VETx, U3 74LVC574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

Commit message: Some updates of schematic.
Parts:
- added D1: GREEN, symbol Device:LED_ALT
- added D2: RED, symbol Device:LED_ALT
- added D3: YELLOW, symbol Device:LED_ALT
- added J6: 4P4C, symbol Connector:4P4C
- added R13, R14, R15: 330, symbol Device:R_Small
Connections:
- net labels added: GREEN, RED, SCL, SDA, YELLOW
- wire segments 420 -> 439
- no-connect marks 41 -> 37
Changed lines of the file:
@@
-DATA_FLG
-Wire Wire Line
-	5450 8700 5800 8700
-Text Label 5500 8700 0    50   ~ 0
 DATA_FLG
 Wire Wire Line
@@
 	4500 4900 4100 4900
 Text Label 4100 4900 0    50   ~ 0
-DATA_FLG
+DATACLK
 $Comp
 L power:+5V #PWR0101
@@
 NoConn ~ 6300 4300
 NoConn ~ 6300 4200
-NoConn ~ 6300 4100
-NoConn ~ 6300 4000
-NoConn ~ 6300 3900
-NoConn ~ 6300 3800
-NoConn ~ 6300 3700
 NoConn ~ 6300 3600
 NoConn ~ 6300 3500
@@
 Wire Wire Line
 	12100 1950 12500 1950
-Wire Wire Line
-	800  2050 1450 2050
-Wire Bus Line
-	2450 3150 2450 3650
-Wire Bus Line
-	7800 3850 7800 4500
-Wire Bus Line
-	2550 1950 2550 3150
-Wire Bus Line
-	700  1950 700  3900
-Wire Bus Line
-	6750 4500 6750 4800
-Wire Bus Line
-	9400 3200 9400 6800
-Wire Bus Line
-	12600 3200 12600 5650
-Wire Bus Line
-	11050 3200 11050 5650
-Wire Bus Line
-	11050 5650 11050 7300
-Wire Bus Line
-	9050 1250 9050 2650
-Wire Bus Line
-	10950 600  10950 1650
-Wire Bus Line
-	950  2050 950  3650
-Wire Bus Line
-	2450 2250 2450 3050
-Wire Bus Line
-	8800 600  8800 1750
-Wire Bus Line
-	6900 1250 6900 2650
-Wire Bus Line
-	9600 2750 9600 6950
-Wire Bus Line
-	6750 1300 6750 2750
-Wire Bus Line
-	4050 600  4050 4300
 Connection ~ 12500 1950
 Wire Wire Line
@@
 	1    0    0    -1
 $EndComp
+Wire Wire Line
+	6300 3700 6650 3700
+Wire Wire Line
+	6300 3800 6650 3800
+Text Label 6400 3700 0    50   ~ 0
+SCL
+Text Label 6400 3800 0    50   ~ 0
+SDA
+$Comp
+L Connector:4P4C J6
+U 1 1 62E2EC2B
+P 7050 7950
+F 0 "J6" H 7105 8417 50  0000 C CNN
+F 1 "4P4C" H 7105 8326 50  0000 C CNN
+F 2 "" V 7050 8000 50  0001 C CNN
+F 3 "~" V 7050 8000 50  0001 C CNN
+	1    7050 7950
+	1    0    0    -1
+$EndComp
+Wire Wire Line
+	7450 7850 7850 7850
+Wire Wire Line
+	7450 7950 7850 7950
+$Comp
+L power:+5V #PWR029
+U 1 1 62EB7006
+P 7550 7650
+F 0 "#PWR029" H 7550 7500 50  0001 C CNN
+F 1 "+5V" H 7565 7823 50  0000 C CNN
+F 2 "" H 7550 7650 50  0001 C CNN
+F 3 "" H 7550 7650 50  0001 C CNN
+	1    7550 7650
+	1    0    0    -1
+$EndComp
+$Comp
+L power:GND #PWR030
+U 1 1 62EB72F6
+P 7550 8150
+F 0 "#PWR030" H 7550 7900 50  0001 C CNN
+F 1 "GND" H 7555 7977 50  0000 C CNN
+F 2 "" H 7550 8150 50  0001 C CNN
+F 3 "" H 7550 8150 50  0001 C CNN
+	1    7550 8150
+	1    0    0    -1
+$EndComp
+Wire Wire Line
+	7450 8050 7550 8050
+Wire Wire Line
+	7550 8050 7550 8150
+Wire Wire Line
+	7450 7750 7550 7750
+Wire Wire Line
+	7550 7750 7550 7650
+Text Label 7650 7850 0    50   ~ 0
+SCL
+Text Label 7650 7950 0    50   ~ 0
+SDA
+$Comp
+L Device:LED_ALT D1
+U 1 1 62F42340
+P 14450 2750
+F 0 "D1" H 14442 2495 50  0000 C CNN
+F 1 "GREEN" H 14442 2586 50  0000 C CNN
+F 2 "" H 14450 2750 50  0001 C CNN
+F 3 "~" H 14450 2750 50  0001 C CNN
+	1    14450 2750
+	-1   0    0    1
+$EndComp
+$Comp
+L Device:LED_ALT D2
+U 1 1 62F42686
+P 14450 3150
+F 0 "D2" H 14442 2895 50  0000 C CNN
+F 1 "RED" H 14442 2986 50  0000 C CNN
+F 2 "" H 14450 3150 50  0001 C CNN
+F 3 "~" H 14450 3150 50  0001 C CNN
+	1    14450 3150
+	-1   0    0    1
+$EndComp
+$Comp
+L Device:LED_ALT D3
+U 1 1 62F42843
+P 14450 3550
+F 0 "D3" H 14442 3295 50  0000 C CNN
+F 1 "YELLOW" H 14442 3386 50  0000 C CNN
+F 2 "" H 14450 3550 50  0001 C CNN
+F 3 "~" H 14450 3550 50  0001 C CNN
+	1    14450 3550
+	-1   0    0    1
+$EndComp
+$Comp
+L Device:R_Small R13
+U 1 1 62F42AFE
+P 13950 2750
+F 0 "R13" V 13754 2750 50  0000 C CNN
+F 1 "330" V 13845 2750 50  0000 C CNN
+F 2 "" H 13950 2750 50  0001 C CNN
+F 3 "~" H 13950 2750 50  0001 C CNN
+	1    13950 2750
+	0    1    1    0
+$EndComp
+$Comp
+L Device:R_Small R14
+U 1 1 62F42D5F
+P 13950 3150
+F 0 "R14" V 13754 3150 50  0000 C CNN
+F 1 "330" V 13845 3150 50  0000 C CNN
+F 2 "" H 13950 3150 50  0001 C CNN
+F 3 "~" H 13950 3150 50  0001 C CNN
+	1    13950 3150
+	0    1    1    0
+$EndComp
+$Comp
+L Device:R_Small R15
+U 1 1 62F42E23
+P 13950 3550
+F 0 "R15" V 13754 3550 50  0000 C CNN
+F 1 "330" V 13845 3550 50  0000 C CNN
+F 2 "" H 13950 3550 50  0001 C CNN
+F 3 "~" H 13950 3550 50  0001 C CNN
+	1    13950 3550
+	0    1    1    0
+$EndComp
+Wire Wire Line
+	14050 2750 14300 2750
+Wire Wire Line
+	14050 3150 14300 3150
+Wire Wire Line
+	14050 3550 14300 3550
+Wire Wire Line
+	14600 2750 14900 2750
+Wire Wire Line
+	14600 3150 14900 3150
+Wire Wire Line
+	14600 3550 14900 3550
+Wire Wire Line
+	13850 3550 13850 3150
+Connection ~ 13850 2750
+Wire Wire Line
+	13850 2750 13850 2350
+Connection ~ 13850 3150
+Wire Wire Line
+	13850 3150 13850 2750
+$Comp
+L power:+3.3V #PWR031
+U 1 1 63174BC3
+P 13850 2350
+F 0 "#PWR031" H 13850 2200 50  0001 C CNN
+F 1 "+3.3V" H 13865 2523 50  0000 C CNN
+F 2 "" H 13850 2350 50  0001 C CNN
+F 3 "" H 13850 2350 50  0001 C CNN
+	1    13850 2350
+	1    0    0    -1
+$EndComp
+Text Label 14650 2750 0    50   ~ 0
+GREEN
+Text Label 14650 3150 0    50   ~ 0
+RED
+Text Label 14650 3550 0    50   ~ 0
+YELLOW
+Wire Wire Line
+	6300 3900 6650 3900
+Wire Wire Line
+	6300 4000 6650 4000
+Wire Wire Line
+	6300 4100 6650 4100
+Text Label 6350 3900 0    50   ~ 0
+RED
+Text Label 6350 4000 0    50   ~ 0
+GREEN
+Text Label 6350 4100 0    50   ~ 0
+YELLOW
+NoConn ~ 5450 8700
+Wire Wire Line
+	800  2050 1450 2050
+Wire Bus Line
+	2450 3150 2450 3650
+Wire Bus Line
+	7800 3850 7800 4500
+Wire Bus Line
+	2550 1950 2550 3150
+Wire Bus Line
+	700  1950 700  3900
+Wire Bus Line
+	6750 4500 6750 4800
+Wire Bus Line
+	9400 3200 9400 6800
+Wire Bus Line
+	12600 3200 12600 5650
+Wire Bus Line
+	11050 3200 11050 5650
+Wire Bus Line
+	11050 5650 11050 7300
+Wire Bus Line
+	9050 1250 9050 2650
+Wire Bus Line
+	10950 600  10950 1650
+Wire Bus Line
+	950  2050 950  3650
+Wire Bus Line
+	2450 2250 2450 3050
+Wire Bus Line
+	8800 600  8800 1750
+Wire Bus Line
+	6900 1250 6900 2650
+Wire Bus Line
+	9600 2750 9600 6950
+Wire Bus Line
+	6750 1300 6750 2750
+Wire Bus Line
+	4050 600  4050 4300
 $EndSCHEMATC
